Commit message: enable velodyne and disable ur5e

File: raigor/raigor_description/urdf/xacro/main.xacro (robot description, xacro)
@@ -1,15 +1,15 @@
 <?xml version="1.0"?>
-<robot xmlns:xacro="http://www.ros.org/wiki/xacro" name="raigor" >
-    <!-- <xacro:arg name="gpu" default="true"/>
+<robot xmlns:xacro="http://www.ros.org/wiki/xacro" name="raigor">
+    <xacro:arg name="gpu" default="true" />
     <xacro:property name="gpu" value="$(arg gpu)" />
-    <xacro:arg name="organize_cloud" default="true"/>
-    <xacro:property name="organize_cloud" value="$(arg organize_cloud)" /> -->
+    <xacro:arg name="organize_cloud" default="true" />
+    <xacro:property name="organize_cloud" value="$(arg organize_cloud)" />
     <xacro:include filename="$(find raigor_description)/urdf/xacro/common.gazebo.xacro" />
-    <xacro:include filename="$(find raigor_description)/urdf/xacro/ur5e.urdf.xacro" />
+    <!-- <xacro:include filename="$(find raigor_description)/urdf/xacro/ur5e.urdf.xacro" /> -->
     <xacro:include filename="$(find raigor_description)/urdf/xacro/tracked_vehicle.urdf.xacro" />
     <!-- <xacro:include filename="$(find raigor_description)/urdf/xacro/camera.xacro" /> -->
-    <!-- <xacro:include filename="$(find raigor_description)/urdf/xacro/lidar.xacro" /> -->
+    <xacro:include filename="$(find raigor_description)/urdf/xacro/lidar.xacro" />
     <!-- <xacro:include filename="$(find raigor_description)/urdf/xacro/imu.xacro" /> -->
-    <xacro:include filename="$(find raigor_description)/urdf/xacro/laser_sensor.xacro" />
+    <!-- <xacro:include filename="$(find raigor_description)/urdf/xacro/laser_sensor.xacro" /> -->
     <xacro:property name="manipulator_offset_x" value="0.365" />
     <xacro:property name="manipulator_offset_y" value="0" />
@@ -21,6 +21,6 @@
     <xacro:property name="lidar_offset_y" value="0" />
     <xacro:property name="lidar_offset_z" value="0.33" /> -->
-    <xacro:d435_gazebo />
-    <xacro:ur5e_robot prefix="" joint_limited="false"
+    <!-- <xacro:d435_gazebo /> -->
+    <!-- <xacro:ur5e_robot prefix="" joint_limited="false"
         shoulder_pan_lower_limit="${-2.0*pi}" shoulder_pan_upper_limit="${2.0*pi}"
         shoulder_lift_lower_limit="${-2.0*pi}" shoulder_lift_upper_limit="${2.0*pi}"
@@ -28,5 +28,5 @@
         wrist_1_lower_limit="${-2.0*pi}" wrist_1_upper_limit="${2.0*pi}"
         wrist_2_lower_limit="${-2.0*pi}" wrist_2_upper_limit="${2.0*pi}"
-        wrist_3_lower_limit="${-2.0*pi}" wrist_3_upper_limit="${2.0*pi}"/>
+        wrist_3_lower_limit="${-2.0*pi}" wrist_3_upper_limit="${2.0*pi}" /> -->
     <!-- <xacro:usb_camera prefix="usb_camera"/> -->
     <link name="board_link">
@@ -43,5 +43,5 @@
         </collision>
     </link>
-<!--
+    <!--
     <link name="support_link">
         <origin xyz="0.0 0.0 0.0" rpy="0 0 0" />
@@ -80,11 +80,11 @@
     <joint name="base_footprint_joint" type="fixed">
         <origin xyz="0 0 0" rpy="0 0 0" />
-        <parent link="base_footprint"/>
+        <parent link="base_footprint" />
         <child link="vehicle_base_link" />
     </joint>
     <joint name="board_joint" type="fixed">
         <origin xyz="-0.055 0 0.32" rpy="0 0 0" />
-        <parent link="vehicle_base_link"/>
-        <child link="board_link"/>
+        <parent link="vehicle_base_link" />
+        <child link="board_link" />
     </joint>
     <!-- <joint name="support_joint" type="fixed">
@@ -95,17 +95,18 @@
     <joint name="lidar_support_joint" type="fixed">
         <origin xyz="-0.05 0.0 0.48" rpy="0 0 0" />
-        <parent link="vehicle_base_link"/>
-        <child link="lidar_support_link"/>
+        <parent link="vehicle_base_link" />
+        <child link="lidar_support_link" />
     </joint>
-    <!-- <xacro:velodyne parent="lidar_support_link" name="velodyne" topic="/velodyne_points" organize_cloud="${organize_cloud}" hz="10" samples="220" gpu="${gpu}">
+    <xacro:velodyne parent="lidar_support_link" name="velodyne" topic="/velodyne_points"
+        organize_cloud="${organize_cloud}" hz="10" samples="220" gpu="${gpu}">
         <origin xyz="0.0 0 0.0" rpy="0 0 0" />
-    </xacro:velodyne> -->
+    </xacro:velodyne>
     <!-- <xacro:imu/> -->
-    <xacro:rplidar/>
+    <!-- <xacro:rplidar />
     <joint name="laser_support_joint" type="fixed">
         <origin xyz="0.0 0.0 0.02" rpy="0 0 0" />
-        <parent link="lidar_support_link"/>
-        <child link="laser_link"/>
-    </joint>
+        <parent link="lidar_support_link" />
+        <child link="laser_link" />
+    </joint> -->
     <!-- <joint name="camera_support_joint" type="fixed">
         <origin xyz="0.30  0  0.50" rpy="0 0 0" />
@@ -118,20 +119,21 @@
         <child link="imu_link"/>
     </joint> -->
-    <joint name="associate_joint" type="fixed">
-        <origin xyz="${manipulator_offset_x} ${manipulator_offset_y} ${manipulator_offset_z}" rpy="0 0 0" />
-        <parent link="vehicle_base_link"/>
-        <child link="base_link"/>
-    </joint>
+    <!-- <joint name="associate_joint" type="fixed">
+        <origin xyz="${manipulator_offset_x} ${manipulator_offset_y} ${manipulator_offset_z}"
+            rpy="0 0 0" />
+        <parent link="vehicle_base_link" />
+        <child link="base_link" />
+    </joint> -->
     <gazebo>
-      <plugin name="p3d_base_controller" filename="libgazebo_ros_p3d.so">
-        <alwaysOn>true</alwaysOn>
-        <updateRate>100.0</updateRate>
-        <bodyName>base_footprint</bodyName>
-        <topicName>base_pose_ground_truth</topicName>
-        <gaussianNoise>0.0</gaussianNoise>
-        <frameName>map</frameName>
-        <xyzOffsets>0 0 0</xyzOffsets>
-        <rpyOffsets>0 0 0</rpyOffsets>
-      </plugin>
+        <plugin name="p3d_base_controller" filename="libgazebo_ros_p3d.so">
+            <alwaysOn>true</alwaysOn>
+            <updateRate>100.0</updateRate>
+            <bodyName>base_footprint</bodyName>
+            <topicName>base_pose_ground_truth</topicName>
+            <gaussianNoise>0.0</gaussianNoise>
+            <frameName>map</frameName>
+            <xyzOffsets>0 0 0</xyzOffsets>
+            <rpyOffsets>0 0 0</rpyOffsets>
+        </plugin>
     </gazebo>
 </robot>
